Commit message: v2

File: lidar_bot_description/gazebo/lidar-bot.gazebo.xacro (robot description, xacro)
@@ -1,9 +1,9 @@
 <?xml version="1.0"?>
 <robot xmlns:xacro="http://ros.org/wiki/xacro">
-  <xacro:macro name="lidar-bot_gazebo">
+  <xacro:macro name="lidar_bot_gazebo">
     <!-- =============== Gazebo =============== -->
     <gazebo>
       <plugin filename="gz_ros2_control-system" name="gz_ros2_control::GazeboSimROS2ControlPlugin">
-        <parameters>$(find lidar-bot_description)/config/lidar-bot_sim.yaml</parameters>
+        <parameters>$(find lidar_bot_description)/config/lidar_bot_sim.yaml</parameters>
       </plugin>
       <plugin filename="gz-sim-sensors-system" name="gz::sim::systems::Sensors">

File: lidar_bot_description/robots/lidar-bot.urdf.xacro (robot description, xacro)
@@ -1,12 +1,12 @@
 <?xml version="1.0"?>
 <!-- Basic differential drive mobile base -->
-<robot xmlns:xacro="http://www.ros.org/wiki/xacro" name="lidar-bot">
-  <xacro:include filename="$(find lidar-bot_description)/gazebo/lidar-bot.gazebo.xacro" />
-  <xacro:include filename="$(find lidar-bot_description)/ros2_control/lidar-bot.ros2_control.xacro" />
-  <xacro:include filename="$(find lidar-bot_description)/robots/parts/base/base.urdf.xacro"/>
-  <xacro:include filename="$(find lidar-bot_description)/robots/parts/suspension/suspension.urdf.xacro"/>
-  <xacro:include filename="$(find lidar-bot_description)/robots/parts/wheel/wheel.urdf.xacro"/>
-  <xacro:include filename="$(find lidar-bot_description)/robots/parts/lidar_base/lidar_base.urdf.xacro"/>
-  <xacro:include filename="$(find lidar-bot_description)/robots/parts/lidar_head/lidar_head.urdf.xacro"/>
+<robot xmlns:xacro="http://www.ros.org/wiki/xacro" name="lidar_bot">
+  <xacro:include filename="$(find lidar_bot_description)/gazebo/lidar_bot.gazebo.xacro" />
+  <xacro:include filename="$(find lidar_bot_description)/ros2_control/lidar_bot.ros2_control.xacro" />
+  <xacro:include filename="$(find lidar_bot_description)/robots/parts/base/base.urdf.xacro"/>
+  <xacro:include filename="$(find lidar_bot_description)/robots/parts/suspension/suspension.urdf.xacro"/>
+  <xacro:include filename="$(find lidar_bot_description)/robots/parts/wheel/wheel.urdf.xacro"/>
+  <xacro:include filename="$(find lidar_bot_description)/robots/parts/lidar_base/lidar_base.urdf.xacro"/>
+  <xacro:include filename="$(find lidar_bot_description)/robots/parts/lidar_head/lidar_head.urdf.xacro"/>
   <xacro:property name="M_PI" value="3.14159274"/>
   <material name="gray">
@@ -89,5 +89,5 @@
   <xacro:steering_gazebo_v0 prefix="rear_right"/>
   <xacro:steering_gazebo_v0 prefix="rear_left"/>
-  <xacro:lidar-bot_gazebo/>
-  <xacro:lidar-bot_ros2_control/>
+  <xacro:lidar_bot_gazebo/>
+  <xacro:lidar_bot_ros2_control/>
 </robot>

File: lidar_bot_description/robots/parts/base/base.urdf.xacro (robot description, xacro)
@@ -1,5 +1,5 @@
 <?xml version="1.0"?>
 <robot xmlns:xacro="http://ros.org/wiki/xacro">
-  <xacro:include filename="$(find lidar-bot_description)/robots/parts/base/base.gazebo.xacro"/>
+  <xacro:include filename="$(find lidar_bot_description)/robots/parts/base/base.gazebo.xacro"/>
   <xacro:macro name="base_v0" params="parent *joint_origin">
 	<joint name="base_link_joint" type="fixed">
@@ -11,10 +11,10 @@
 	  <visual>
 		<geometry>
-		  <mesh filename="package://lidar-bot_description/meshes/DAE/base/base_link.dae"/>
+		  <mesh filename="package://lidar_bot_description/meshes/DAE/base/base_link.dae"/>
 		</geometry>
 	  </visual>
 	  <collision>
 		<geometry>
-		  <mesh filename="package://lidar-bot_description/meshes/STL/base/base_link.stl"/>
+		  <mesh filename="package://lidar_bot_description/meshes/STL/base/base_link.stl"/>
 		</geometry>
 	  </collision>

File: lidar_bot_description/robots/parts/lidar_base/lidar_base.urdf.xacro (robot description, xacro)
@@ -1,5 +1,5 @@
 <?xml version="1.0"?>
 <robot xmlns:xacro="http://ros.org/wiki/xacro">
-  <xacro:include filename="$(find lidar-bot_description)/robots/parts/lidar_base/lidar_base.gazebo.xacro"/>
+  <xacro:include filename="$(find lidar_bot_description)/robots/parts/lidar_base/lidar_base.gazebo.xacro"/>
   <xacro:macro name="lidar_base_v0" params="parent *joint_origin">
 	<joint name="lidar_base_link_joint" type="fixed">
@@ -11,10 +11,10 @@
 	  <visual>
 		<geometry>
-		  <mesh filename="package://lidar-bot_description/meshes/DAE/lidar_base/YDlidar_base.dae"/>
+		  <mesh filename="package://lidar_bot_description/meshes/DAE/lidar_base/YDlidar_base.dae"/>
 		</geometry>
 	  </visual>
 	  <collision>
 		<geometry>
-		  <mesh filename="package://lidar-bot_description/meshes/STL/lidar_base/YDlidar_base.stl"/>
+		  <mesh filename="package://lidar_bot_description/meshes/STL/lidar_base/YDlidar_base.stl"/>
 		</geometry>
 	  </collision>

File: lidar_bot_description/robots/parts/lidar_head/lidar_head.urdf.xacro (robot description, xacro)
@@ -1,5 +1,5 @@
 <?xml version="1.0"?>
 <robot xmlns:xacro="http://ros.org/wiki/xacro">
-  <xacro:include filename="$(find lidar-bot_description)/robots/parts/lidar_head/lidar_head.gazebo.xacro"/>
+  <xacro:include filename="$(find lidar_bot_description)/robots/parts/lidar_head/lidar_head.gazebo.xacro"/>
   <xacro:macro name="lidar_head_v0" params="parent *joint_origin">
 	<joint name="lidar_head_joint" type="fixed">
@@ -11,10 +11,10 @@
 	  <visual>
 		<geometry>
-		  <mesh filename="package://lidar-bot_description/meshes/DAE/lidar_head/YDlidar_head.dae"/>
+		  <mesh filename="package://lidar_bot_description/meshes/DAE/lidar_head/YDlidar_head.dae"/>
 		</geometry>
 	  </visual>
 	  <collision>
 		<geometry>
-		  <mesh filename="package://lidar-bot_description/meshes/STL/lidar_head/YDlidar_head.stl"/>
+		  <mesh filename="package://lidar_bot_description/meshes/STL/lidar_head/YDlidar_head.stl"/>
 		</geometry>
 	  </collision>

File: lidar_bot_description/robots/parts/suspension/suspension.urdf.xacro (robot description, xacro)
@@ -1,5 +1,5 @@
 <?xml version="1.0"?>
 <robot xmlns:xacro="http://ros.org/wiki/xacro">
-  <xacro:include filename="$(find lidar-bot_description)/robots/parts/suspension/suspension.gazebo.xacro"/>
+  <xacro:include filename="$(find lidar_bot_description)/robots/parts/suspension/suspension.gazebo.xacro"/>
   <xacro:macro name="steering_v0" params="prefix parent *joint_origin *joint_axis">
 	<joint name="${prefix}_steering_joint" type="revolute">
@@ -13,10 +13,10 @@
 	  <visual>
 		<geometry>
-		  <mesh filename="package://lidar-bot_description/meshes/DAE/suspension/${prefix}_link.dae"/>
+		  <mesh filename="package://lidar_bot_description/meshes/DAE/suspension/${prefix}_link.dae"/>
 		</geometry>
 	  </visual>
 	  <collision>
 		<geometry>
-		  <mesh filename="package://lidar-bot_description/meshes/STL/suspension/sus_link.stl"/>
+		  <mesh filename="package://lidar_bot_description/meshes/STL/suspension/sus_link.stl"/>
 		</geometry>
 	  </collision>

File: lidar_bot_description/robots/parts/wheel/wheel.urdf.xacro (robot description, xacro)
@@ -1,5 +1,5 @@
 <?xml version="1.0"?>
 <robot xmlns:xacro="http://ros.org/wiki/xacro">
-  <xacro:include filename="$(find lidar-bot_description)/robots/parts/wheel/wheel.gazebo.xacro"/>
+  <xacro:include filename="$(find lidar_bot_description)/robots/parts/wheel/wheel.gazebo.xacro"/>
   <xacro:macro name="wheel_v0" params="prefix parent *joint_origin *joint_axis">
 	<joint name="${prefix}_wheel_joint" type="continuous">
@@ -13,10 +13,10 @@
 	  <visual>
 		<geometry>
-		  <mesh filename="package://lidar-bot_description/meshes/DAE/wheel/wheel_link.dae"/>
+		  <mesh filename="package://lidar_bot_description/meshes/DAE/wheel/wheel_link.dae"/>
 		</geometry>
 	  </visual>
 	  <collision>
 		<geometry>
-		  <mesh filename="package://lidar-bot_description/meshes/STL/wheel/robot_wheel.stl"/>
+		  <mesh filename="package://lidar_bot_description/meshes/STL/wheel/robot_wheel.stl"/>
 		</geometry>
 	  </collision>

File: lidar_bot_description/ros2_control/lidar-bot.ros2_control.xacro (robot description, xacro)
@@ -1,5 +1,5 @@
 <?xml version="1.0"?>
 <robot xmlns:xacro="http://www.ros.org/wiki/xacro">
-  <xacro:macro name="lidar-bot_ros2_control">
+  <xacro:macro name="lidar_bot_ros2_control">
     <ros2_control name="fws" type="system">
       <hardware>
